Commit message: push joystick not working

File: src/spongebob_description/urdf/spongebob.xacro (robot description, xacro)
@@ -46,24 +46,4 @@
     <child link="base_footprint"/>
     <origin xyz="${base_length/2} 0.0 0.0" rpy="0 0 0"/>
-  </joint>
-  <link name="marking_base"/>
-  <joint name="marking_base_joint" type="fixed">
-    <parent link="marking_base"/>
-    <child link="base_link"/>
-    <origin xyz="0.0 0.0 0.0" rpy="0 0 0"/>
-  </joint>
-  <link name="marking_spot">
-    <visual>
-      <geometry>
-        <cylinder radius="0.01" length="0.001"/>
-      </geometry>
-      <origin xyz="0 0 0" rpy="0 0 0"/>
-      <material name="red"/>
-    </visual>
-  </link>
-  <joint name="marking_joint" type="fixed">
-    <parent link="marking_spot"/>
-    <child link="marking_base"/>
-    <origin xyz="0.0 0.0 0.0" rpy="0 0 0"/>
   </joint>
   <link name="caster">
